Commit message: Add FRI port number to urdf

File: robots/iiwa.urdf.xacro (robot description, xacro)
@@ -4,4 +4,5 @@
   <xacro:arg name="prefix" default="$(arg robot)_"/>
   <xacro:arg name="robot_ip" default="192.170.10.1"/>
+  <xacro:arg name="fri_port" default="30200"/>
   <xacro:arg name="load_ros2_control" default="false"/>
   <xacro:arg name="use_sim" default="false"/>
@@ -22,5 +23,5 @@
   <xacro:if value="$(arg load_ros2_control)">
     <xacro:iiwa_interface name="IiwaInterface" prefix="$(arg prefix)" robot_ip="$(arg robot_ip)"
-                          use_sim="$(arg use_sim)"/>
+                          fri_port="${arg fri_port}" use_sim="$(arg use_sim)"/>
   </xacro:if>
 </robot>

File: ros2_control/iiwa.ros2_control.xacro (robot description, xacro)
@@ -1,5 +1,5 @@
 <?xml version="1.0"?>
 <robot xmlns:xacro="http://www.ros.org/wiki/xacro">
-  <xacro:macro name="iiwa_interface" params="name prefix robot_ip use_sim">
+  <xacro:macro name="iiwa_interface" params="name prefix robot_ip fri_port use_sim">
     <ros2_control name="${name}" type="system">
       <xacro:unless value="${use_sim}">
@@ -7,4 +7,5 @@
           <plugin>robot_interface/iiwa/IiwaInterface</plugin>
           <param name="robot_ip">${robot_ip}</param>
+          <param name="fri_port">${fri_port}</param>
         </hardware>
       </xacro:unless>

Commit message: Rename fri port to port

File: robots/iiwa.urdf.xacro (robot description, xacro)
@@ -4,5 +4,5 @@
   <xacro:arg name="prefix" default="$(arg robot)_"/>
   <xacro:arg name="robot_ip" default="192.170.10.1"/>
-  <xacro:arg name="fri_port" default="30200"/>
+  <xacro:arg name="port" default="30200"/>
   <xacro:arg name="load_ros2_control" default="false"/>
   <xacro:arg name="use_sim" default="false"/>
@@ -24,5 +24,5 @@
     <xacro:include filename="$(find kuka_iiwa_description)/ros2_control/iiwa.ros2_control.xacro"/>
     <xacro:iiwa_interface name="IiwaInterface" prefix="$(arg prefix)" robot_ip="$(arg robot_ip)"
-                          fri_port="$(arg fri_port)" use_sim="$(arg use_sim)"/>
+                          port="$(arg port)" use_sim="$(arg use_sim)"/>
   </xacro:if>
 </robot>

File: ros2_control/iiwa.ros2_control.xacro (robot description, xacro)
@@ -1,5 +1,5 @@
 <?xml version="1.0"?>
 <robot xmlns:xacro="http://www.ros.org/wiki/xacro">
-  <xacro:macro name="iiwa_interface" params="name prefix robot_ip fri_port use_sim">
+  <xacro:macro name="iiwa_interface" params="name prefix robot_ip port use_sim">
     <ros2_control name="${name}" type="system">
       <xacro:unless value="${use_sim}">
@@ -7,5 +7,5 @@
           <plugin>robot_interface/kuka/IiwaInterface</plugin>
           <param name="robot_ip">${robot_ip}</param>
-          <param name="fri_port">${fri_port}</param>
+          <param name="port">${port}</param>
         </hardware>
       </xacro:unless>

Commit message: Add port number and fix bugs (#3)
* Add FRI port number to urdf

* Fix ros2_control macro

* Fix brackets

* Fix wrong minuses

* Rename fri port to port

File: robots/iiwa.urdf.xacro (robot description, xacro)
@@ -4,4 +4,5 @@
   <xacro:arg name="prefix" default="$(arg robot)_"/>
   <xacro:arg name="robot_ip" default="192.170.10.1"/>
+  <xacro:arg name="port" default="30200"/>
   <xacro:arg name="load_ros2_control" default="false"/>
   <xacro:arg name="use_sim" default="false"/>
@@ -21,6 +22,7 @@
   </xacro:if>
   <xacro:if value="$(arg load_ros2_control)">
+    <xacro:include filename="$(find kuka_iiwa_description)/ros2_control/iiwa.ros2_control.xacro"/>
     <xacro:iiwa_interface name="IiwaInterface" prefix="$(arg prefix)" robot_ip="$(arg robot_ip)"
-                          use_sim="$(arg use_sim)"/>
+                          port="$(arg port)" use_sim="$(arg use_sim)"/>
   </xacro:if>
 </robot>

File: ros2_control/iiwa.ros2_control.xacro (robot description, xacro)
@@ -1,10 +1,11 @@
 <?xml version="1.0"?>
 <robot xmlns:xacro="http://www.ros.org/wiki/xacro">
-  <xacro:macro name="iiwa_interface" params="name prefix robot_ip use_sim">
+  <xacro:macro name="iiwa_interface" params="name prefix robot_ip port use_sim">
     <ros2_control name="${name}" type="system">
       <xacro:unless value="${use_sim}">
         <hardware>
-          <plugin>robot_interface/iiwa/IiwaInterface</plugin>
+          <plugin>robot_interface/kuka/IiwaInterface</plugin>
           <param name="robot_ip">${robot_ip}</param>
+          <param name="port">${port}</param>
         </hardware>
       </xacro:unless>
@@ -29,5 +30,5 @@
       <joint name="${prefix}joint2">
         <command_interface name="position">
-          <param name="min">-${-joint_limit_2}</param>
+          <param name="min">${-joint_limit_2}</param>
           <param name="max">${joint_limit_2}</param>
         </command_interface>
@@ -47,5 +48,5 @@
       <joint name="${prefix}joint3">
         <command_interface name="position">
-          <param name="min">-${-joint_limit_3}</param>
+          <param name="min">${-joint_limit_3}</param>
           <param name="max">${joint_limit_3}</param>
         </command_interface>
@@ -65,5 +66,5 @@
       <joint name="${prefix}joint4">
         <command_interface name="position">
-          <param name="min">-${-joint_limit_4}</param>
+          <param name="min">${-joint_limit_4}</param>
           <param name="max">${joint_limit_4}</param>
         </command_interface>
@@ -83,5 +84,5 @@
       <joint name="${prefix}joint5">
         <command_interface name="position">
-          <param name="min">-${-joint_limit_5}</param>
+          <param name="min">${-joint_limit_5}</param>
           <param name="max">${joint_limit_5}</param>
         </command_interface>
@@ -101,5 +102,5 @@
       <joint name="${prefix}joint6">
         <command_interface name="position">
-          <param name="min">-${-joint_limit_6}</param>
+          <param name="min">${-joint_limit_6}</param>
           <param name="max">${joint_limit_6}</param>
         </command_interface>
@@ -119,5 +120,5 @@
       <joint name="${prefix}joint7">
         <command_interface name="position">
-          <param name="min">-${-joint_limit_7}</param>
+          <param name="min">${-joint_limit_7}</param>
           <param name="max">${joint_limit_7}</param>
         </command_interface>

Commit message: Add state and command port to ros2 control macro

File: robots/iiwa.urdf.xacro (robot description, xacro)
@@ -3,6 +3,7 @@
   <xacro:arg name="robot" default="iiwa7"/>
   <xacro:arg name="prefix" default="$(arg robot)_"/>
-  <xacro:arg name="robot_ip" default="192.170.10.1"/>
-  <xacro:arg name="port" default="30200"/>
+  <xacro:arg name="robot_ip" default="127.0.0.1"/>
+  <xacro:arg name="robot_state_port" default="9701"/>
+  <xacro:arg name="robot_command_port" default="9702"/>
   <xacro:arg name="load_ros2_control" default="false"/>
   <xacro:arg name="use_sim" default="false"/>
@@ -24,5 +25,6 @@
     <xacro:include filename="$(find kuka_iiwa_description)/ros2_control/iiwa.ros2_control.xacro"/>
     <xacro:iiwa_interface name="IiwaInterface" prefix="$(arg prefix)" robot_ip="$(arg robot_ip)"
-                          port="$(arg port)" use_sim="$(arg use_sim)"/>
+                          robot_state_port="$(arg robot_state_port)" robot_command_port="$(arg robot_command_port)"
+                          use_sim="$(arg use_sim)"/>
   </xacro:if>
 </robot>

File: ros2_control/iiwa.ros2_control.xacro (robot description, xacro)
@@ -1,5 +1,5 @@
 <?xml version="1.0"?>
 <robot xmlns:xacro="http://www.ros.org/wiki/xacro">
-  <xacro:macro name="iiwa_interface" params="name prefix robot_ip port use_sim">
+  <xacro:macro name="iiwa_interface" params="name prefix robot_ip robot_state_port robot_command_port use_sim">
     <ros2_control name="${name}" type="system">
       <xacro:unless value="${use_sim}">
@@ -7,5 +7,6 @@
           <plugin>robot_interface/kuka/IiwaInterface</plugin>
           <param name="robot_ip">${robot_ip}</param>
-          <param name="port">${port}</param>
+          <param name="robot_state_port">${robot_state_port}</param>
+          <param name="robot_command_port">${robot_command_port}</param>
         </hardware>
       </xacro:unless>
