Commit message: Adapt for lightweight interface (#5)
* Add state and command port to ros2 control macro

* Add pybullet interface if sim

File: ros2_control/iiwa.ros2_control.xacro (robot description, xacro)
@@ -1,11 +1,20 @@
 <?xml version="1.0"?>
 <robot xmlns:xacro="http://www.ros.org/wiki/xacro">
-  <xacro:macro name="iiwa_interface" params="name prefix robot_ip port use_sim">
+  <xacro:macro name="iiwa_interface" params="name prefix robot_ip robot_state_port robot_command_port use_sim">
     <ros2_control name="${name}" type="system">
+      <xacro:if value="${use_sim}">
+        <hardware>
+          <plugin>robot_interface/simulators/PybulletInterface</plugin>
+          <param name="robot_ip">${robot_ip}</param>
+          <param name="robot_state_port">${robot_state_port}</param>
+          <param name="robot_command_port">${robot_command_port}</param>
+        </hardware>
+      </xacro:if>
       <xacro:unless value="${use_sim}">
         <hardware>
           <plugin>robot_interface/kuka/IiwaInterface</plugin>
           <param name="robot_ip">${robot_ip}</param>
-          <param name="port">${port}</param>
+          <param name="robot_state_port">${robot_state_port}</param>
+          <param name="robot_command_port">${robot_command_port}</param>
         </hardware>
       </xacro:unless>
